File: nightliner.kicad_sch (KiCad schematic)
At the start: 81 parts, among them J1 TYPE-C-31-M-12, J2 Battery, J3 Battery, SW1 pinky_top, SW10 inner_home, SW11 pinky_bottom, SW12 ring_bottom, SW13 middle_bottom, SW14 index_bottom, SW15 inner_bottom, SW16 outer_top, SW17 outer_home, SW18 near_thumb, SW19 home_thumb, SW2 ring_top, SW20 far_thumb, SW21 ON_OFF, SW22 RESET, SW3 middle_top, SW4 index_top, SW5 inner_top, SW6 pinky_home, SW7 ring_home, SW8 middle_home, SW9 index_home, U1 holyiot-18010, U2 TVS2200DRV, U3 USBLC6-2SC6, U4 BQ24075RGT, U5 XC6220B331MR

Commit message: feat: add mounting holes, better labels
Parts:
- added H1, H2: Alignmenthole, miro_keyboard:Hole_1mm, symbol Mechanical:MountingHole
- added H3, H4, H5, H6, H7, H8, H9: MountingHole_M3, MountingHole:MountingHole_3.2mm_M3, symbol PCM_SL_Mechanical:MountingHole_M3
Other:
- note added: "Mechanical Components"
Changed lines of the file:
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@@
     (stroke (width 0) (type default))
+  )
+  (rectangle (start 66.04 76.2) (end 110.49 91.44)
+    (stroke (width 0) (type dash))
+    (fill (type none))
   )
   (rectangle (start 16.51 97.79) (end 96.52 194.31)
@@
   )
   (text "Programming Pogo Pins" (at 137.16 166.37 0)
+    (effects (font (size 1.27 1.27)) (justify left bottom))
+  )
+  (text "Mechanical Components" (at 66.04 74.93 0)
     (effects (font (size 1.27 1.27)) (justify left bottom))
   )
@@
         (path "/e4693d91-d111-4059-a601-28406aaad775"
           (reference "SW12") (unit 1)
+        )
+      )
+    )
+  )
+  (symbol (lib_id "PCM_SL_Mechanical:MountingHole_M3") (at 80.01 86.36 0) (unit 1)
+    (in_bom yes) (on_board yes) (dnp no) (fields_autoplaced)
+    (property "Reference" "H8" (at 83.82 86.36 0)
+      (effects (font (size 1.27 1.27)) (justify left))
+    )
+    (property "Value" "MountingHole_M3" (at 83.82 87.63 0)
+      (effects (font (size 1.27 1.27)) (justify left) hide)
+    )
+    (property "Footprint" "MountingHole:MountingHole_3.2mm_M3" (at 80.01 90.17 0)
+      (effects (font (size 1.27 1.27)) hide)
+    )
+    (property "Datasheet" "" (at 80.01 86.36 0)
+      (effects (font (size 1.27 1.27)) hide)
+    )
+    (instances
+      (project "nightliner"
+        (path "/e4693d91-d111-4059-a601-28406aaad775"
+          (reference "H8") (unit 1)
         )
       )
@@
     )
   )
+  (symbol (lib_id "Mechanical:MountingHole") (at 154.94 173.99 0) (unit 1)
+    (in_bom yes) (on_board yes) (dnp no) (fields_autoplaced)
+    (property "Reference" "H2" (at 157.48 173.99 0)
+      (effects (font (size 1.27 1.27)) (justify left))
+    )
+    (property "Value" "Alignmenthole" (at 157.48 175.26 0)
+      (effects (font (size 1.27 1.27)) (justify left) hide)
+    )
+    (property "Footprint" "miro_keyboard:Hole_1mm" (at 154.94 173.99 0)
+      (effects (font (size 1.27 1.27)) hide)
+    )
+    (property "Datasheet" "~" (at 154.94 173.99 0)
+      (effects (font (size 1.27 1.27)) hide)
+    )
+    (instances
+      (project "nightliner"
+        (path "/e4693d91-d111-4059-a601-28406aaad775"
+          (reference "H2") (unit 1)
+        )
+      )
+    )
+  )
   (symbol (lib_id "Device:C") (at 270.51 128.27 0) (unit 1)
     (in_bom yes) (on_board yes) (dnp no)
@@
     )
   )
+  (symbol (lib_id "PCM_SL_Mechanical:MountingHole_M3") (at 90.17 80.01 0) (unit 1)
+    (in_bom yes) (on_board yes) (dnp no) (fields_autoplaced)
+    (property "Reference" "H5" (at 93.98 80.01 0)
+      (effects (font (size 1.27 1.27)) (justify left))
+    )
+    (property "Value" "MountingHole_M3" (at 93.98 81.28 0)
+      (effects (font (size 1.27 1.27)) (justify left) hide)
+    )
+    (property "Footprint" "MountingHole:MountingHole_3.2mm_M3" (at 90.17 83.82 0)
+      (effects (font (size 1.27 1.27)) hide)
+    )
+    (property "Datasheet" "" (at 90.17 80.01 0)
+      (effects (font (size 1.27 1.27)) hide)
+    )
+    (instances
+      (project "nightliner"
+        (path "/e4693d91-d111-4059-a601-28406aaad775"
+          (reference "H5") (unit 1)
+        )
+      )
+    )
+  )
   (symbol (lib_id "Device:R") (at 191.77 113.03 90) (unit 1)
     (in_bom yes) (on_board yes) (dnp no)
@@
         (path "/e4693d91-d111-4059-a601-28406aaad775"
           (reference "SW8") (unit 1)
+        )
+      )
+    )
+  )
+  (symbol (lib_id "PCM_SL_Mechanical:MountingHole_M3") (at 69.85 80.01 0) (unit 1)
+    (in_bom yes) (on_board yes) (dnp no) (fields_autoplaced)
+    (property "Reference" "H3" (at 73.66 80.01 0)
+      (effects (font (size 1.27 1.27)) (justify left))
+    )
+    (property "Value" "MountingHole_M3" (at 73.66 81.28 0)
+      (effects (font (size 1.27 1.27)) (justify left) hide)
+    )
+    (property "Footprint" "MountingHole:MountingHole_3.2mm_M3" (at 69.85 83.82 0)
+      (effects (font (size 1.27 1.27)) hide)
+    )
+    (property "Datasheet" "" (at 69.85 80.01 0)
+      (effects (font (size 1.27 1.27)) hide)
+    )
+    (instances
+      (project "nightliner"
+        (path "/e4693d91-d111-4059-a601-28406aaad775"
+          (reference "H3") (unit 1)
         )
       )
@@
         (path "/e4693d91-d111-4059-a601-28406aaad775"
           (reference "J3") (unit 1)
+        )
+      )
+    )
+  )
+  (symbol (lib_id "PCM_SL_Mechanical:MountingHole_M3") (at 90.17 86.36 0) (unit 1)
+    (in_bom yes) (on_board yes) (dnp no) (fields_autoplaced)
+    (property "Reference" "H9" (at 93.98 86.36 0)
+      (effects (font (size 1.27 1.27)) (justify left))
+    )
+    (property "Value" "MountingHole_M3" (at 93.98 87.63 0)
+      (effects (font (size 1.27 1.27)) (justify left) hide)
+    )
+    (property "Footprint" "MountingHole:MountingHole_3.2mm_M3" (at 90.17 90.17 0)
+      (effects (font (size 1.27 1.27)) hide)
+    )
+    (property "Datasheet" "" (at 90.17 86.36 0)
+      (effects (font (size 1.27 1.27)) hide)
+    )
+    (instances
+      (project "nightliner"
+        (path "/e4693d91-d111-4059-a601-28406aaad775"
+          (reference "H9") (unit 1)
         )
       )
@@
     )
   )
+  (symbol (lib_id "PCM_SL_Mechanical:MountingHole_M3") (at 69.85 86.36 0) (unit 1)
+    (in_bom yes) (on_board yes) (dnp no) (fields_autoplaced)
+    (property "Reference" "H7" (at 73.66 86.36 0)
+      (effects (font (size 1.27 1.27)) (justify left))
+    )
+    (property "Value" "MountingHole_M3" (at 73.66 87.63 0)
+      (effects (font (size 1.27 1.27)) (justify left) hide)
+    )
+    (property "Footprint" "MountingHole:MountingHole_3.2mm_M3" (at 69.85 90.17 0)
+      (effects (font (size 1.27 1.27)) hide)
+    )
+    (property "Datasheet" "" (at 69.85 86.36 0)
+      (effects (font (size 1.27 1.27)) hide)
+    )
+    (instances
+      (project "nightliner"
+        (path "/e4693d91-d111-4059-a601-28406aaad775"
+          (reference "H7") (unit 1)
+        )
+      )
+    )
+  )
   (symbol (lib_id "power:GND") (at 246.38 152.4 0) (unit 1)
     (in_bom yes) (on_board yes) (dnp no) (fields_autoplaced)
@@
     )
   )
+  (symbol (lib_id "PCM_SL_Mechanical:MountingHole_M3") (at 100.33 80.01 0) (unit 1)
+    (in_bom yes) (on_board yes) (dnp no) (fields_autoplaced)
+    (property "Reference" "H6" (at 104.14 80.01 0)
+      (effects (font (size 1.27 1.27)) (justify left))
+    )
+    (property "Value" "MountingHole_M3" (at 104.14 81.28 0)
+      (effects (font (size 1.27 1.27)) (justify left) hide)
+    )
+    (property "Footprint" "MountingHole:MountingHole_3.2mm_M3" (at 100.33 83.82 0)
+      (effects (font (size 1.27 1.27)) hide)
+    )
+    (property "Datasheet" "" (at 100.33 80.01 0)
+      (effects (font (size 1.27 1.27)) hide)
+    )
+    (instances
+      (project "nightliner"
+        (path "/e4693d91-d111-4059-a601-28406aaad775"
+          (reference "H6") (unit 1)
+        )
+      )
+    )
+  )
+  (symbol (lib_id "PCM_SL_Mechanical:MountingHole_M3") (at 80.01 80.01 0) (unit 1)
+    (in_bom yes) (on_board yes) (dnp no) (fields_autoplaced)
+    (property "Reference" "H4" (at 83.82 80.01 0)
+      (effects (font (size 1.27 1.27)) (justify left))
+    )
+    (property "Value" "MountingHole_M3" (at 83.82 81.28 0)
+      (effects (font (size 1.27 1.27)) (justify left) hide)
+    )
+    (property "Footprint" "MountingHole:MountingHole_3.2mm_M3" (at 80.01 83.82 0)
+      (effects (font (size 1.27 1.27)) hide)
+    )
+    (property "Datasheet" "" (at 80.01 80.01 0)
+      (effects (font (size 1.27 1.27)) hide)
+    )
+    (instances
+      (project "nightliner"
+        (path "/e4693d91-d111-4059-a601-28406aaad775"
+          (reference "H4") (unit 1)
+        )
+      )
+    )
+  )
   (symbol (lib_id "Device:C") (at 199.39 124.46 0) (unit 1)
     (in_bom yes) (on_board yes) (dnp no)
@@
         )
       )
+    )
+  )
+  (symbol (lib_id "Mechanical:MountingHole") (at 154.94 191.77 0) (unit 1)
+    (in_bom yes) (on_board yes) (dnp no) (fields_autoplaced)
+    (property "Reference" "H1" (at 157.48 191.77 0)
+      (effects (font (size 1.27 1.27)) (justify left))
+    )
+    (property "Value" "Alignmenthole" (at 157.48 193.04 0)
+      (effects (font (size 1.27 1.27)) (justify left) hide)
+    )
+    (property "Footprint" "miro_keyboard:Hole_1mm" (at 154.94 191.77 0)
+      (effects (font (size 1.27 1.27)) hide)
+    )
+    (property "Datasheet" "~" (at 154.94 191.77 0)
+      (effects (font (size 1.27 1.27)) hide)
+    )
+    (instances
+      (project "nightliner"
+        (path "/e4693d91-d111-4059-a601-28406aaad775"
+          (reference "H1") (unit 1)
+        )
+      )

Commit message: feat: change connector and on/off switch, re-layout
Parts:
- J2: footprint Connector_JST:JST_EH_S3B-EH_1x03_P2.50mm_Horizontal -> Connector_JST:JST_XH_S3B-XH-A-1_1x03_P2.50mm_Horizontal
- SW21: footprint miro_keyboard:SW_XKB_SS-12D11_SPDT_Angled -> miro_keyboard:SW_ROCPU_SK-12D07-5_SPDT_Angled
Changed lines of the file:
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@@
       (effects (font (size 1.27 1.27)))
     )
-    (property "Footprint" "miro_keyboard:SW_XKB_SS-12D11_SPDT_Angled" (at 275.59 113.03 0)
+    (property "Footprint" "miro_keyboard:SW_ROCPU_SK-12D07-5_SPDT_Angled" (at 275.59 113.03 0)
       (effects (font (size 1.27 1.27)) hide)
     )
@@
       (effects (font (size 1.27 1.27)) (justify left))
     )
-    (property "Footprint" "Connector_JST:JST_EH_S3B-EH_1x03_P2.50mm_Horizontal" (at 193.04 153.67 0)
+    (property "Footprint" "Connector_JST:JST_XH_S3B-XH-A-1_1x03_P2.50mm_Horizontal" (at 193.04 153.67 0)
       (effects (font (size 1.27 1.27)) hide)
     )

Commit message: fix: footprint for prog header, mounting holes, drc check
Parts:
- removed H1, H2: Alignmenthole, miro_keyboard:Hole_1mm, symbol Mechanical:MountingHole
- removed TP1, TP2, TP3, TP4, TP5: TestPoint, TestPoint:TestPoint_Pad_D1.5mm, symbol Connector:TestPoint
- added P1: ISP_Prog, miro_keyboard:ISP_Programming_Pads, symbol miro_keyboard:ISP_Prog
- D21, D22, D23, D24: footprint Capacitor_SMD:C_0603_1608Metric -> LED_SMD:LED_0603_1608Metric
- F1: footprint Capacitor_SMD:C_0603_1608Metric -> Fuse:Fuse_0603_1608Metric
- H1: renamed from H3; footprint MountingHole:MountingHole_3.2mm_M3 -> MountingHole:MountingHole_6.4mm_M6
- H2: renamed from H6; footprint MountingHole:MountingHole_3.2mm_M3 -> MountingHole:MountingHole_6.4mm_M6
- H3: renamed from H4; footprint MountingHole:MountingHole_3.2mm_M3 -> MountingHole:MountingHole_6.4mm_M6
- H4: renamed from H7; footprint MountingHole:MountingHole_3.2mm_M3 -> MountingHole:MountingHole_6.4mm_M6
- H5: footprint MountingHole:MountingHole_3.2mm_M3 -> MountingHole:MountingHole_6.4mm_M6
- H6: renamed from H8; footprint MountingHole:MountingHole_3.2mm_M3 -> MountingHole:MountingHole_6.4mm_M6
- H7: renamed from H9; footprint MountingHole:MountingHole_3.2mm_M3 -> MountingHole:MountingHole_6.4mm_M6
- U1: footprint kleeb_mcu:holyiot-18010 -> miro_keyboard:holyiot-18010
Connections:
- net GND: now also P1.5 (GND)
- net SWCLK: now also P1.2 (SWCLK)
- net SWDIO: now also P1.3 (SWDIO)
- net SWO: now also P1.4 (SWO)
- net VDD: now also P1.1 (VDD)
Other:
- moved on the sheet: H2, H4, H6, H7
