File: nightliner-left/nightliner.kicad_pcb (KiCad board)
At the start: 2 copper layers, 154.8 x 116.1 mm, 87 parts, among them J1 TYPE-C-31-M-12, J2 Battery, J3 Serial, P1 ISP_Prog, SW1 pinky_top, SW10 inner_home, SW11 pinky_bottom, SW12 ring_bottom, SW13 middle_bottom, SW14 index_bottom, SW15 inner_bottom, SW16 outer_top, SW17 outer_home, SW18 near_thumb, SW19 home_thumb, SW2 ring_top, SW20 far_thumb, SW21 ON_OFF, SW22 RESET, SW3 middle_top, SW4 index_top, SW5 inner_top, SW6 pinky_home, SW7 ring_home, SW8 middle_home, SW9 index_home, U1 holyiot-18010, U2 TVS2200DRV, U3 USBLC6-2SC6, U4 BQ24075RGT, U5 XC6220B331MR

Commit message: fix: rework right case, fix outline
Routing:
- net Net-(D23-K): track 30.1 -> 31.3 mm
- net GND: track 252.0 -> 253.1 mm, vias 17 -> 18

Commit message: fix: final version, create production gerbers
Parts:
- H1, H2, H3, H4, H5, H6, H7: footprint miro_keyboard:StandOff_6mm_M3 -> nightliner:StandOff_6mm_M3
- J3: footprint miro_keyboard:MagConn_6pin_left -> nightliner:MagConn_6pin_left
- P1: footprint miro_keyboard:ISP_Programming_Pads -> nightliner:ISP_Programming_Pads
- SW1, SW10, SW11, SW12, SW13, SW14, SW15, SW16, SW17, SW18, SW19, SW2, SW20, SW3, SW4, SW5, SW6, SW7, SW8, SW9: footprint miro_keyboard:Kailh_Choc_CPG135001D02_Hotswap -> nightliner:Kailh_Choc_CPG135001D02_Hotswap
- SW21: footprint miro_keyboard:SW_ROCPU_SK-12D07-5_SPDT_Angled -> nightliner:SW_ROCPU_SK-12D07-5_SPDT_Angled
- SW22: footprint miro_keyboard:SW_Push_1P1T_NO_CK_KSC4xxJ -> nightliner:SW_Push_1P1T_NO_CK_KSC4xxJ
- U1: footprint miro_keyboard:HOLYIOT-18010-UndersidePins-SMD -> nightliner:HOLYIOT-18010-UndersidePins-SMD
- U4: footprint miro_keyboard:VQFN-16-1EP_3x3mm_P0.5mm_EP1.6x1.6mm_ThermalVias -> nightliner:VQFN-16-1EP_3x3mm_P0.5mm_EP1.6x1.6mm_ThermalVias
- moved H5 6.12 mm to (118.9, 72.1)
- moved H4 3.31 mm to (98.6, 45.7)
Routing:
- net Net-(D16-A): track 148.3 -> 125.1 mm
- net Net-(D11-A): track 108.7 -> 94.7 mm, vias 1 -> 3
- net Net-(D17-A): track 126.4 -> 114.0 mm
- net Net-(D9-A): track 57.9 -> 48.3 mm
- net COL0: track 177.3 -> 168.4 mm
- net Net-(D1-A): track 112.8 -> 121.4 mm
- net Net-(D2-A): track 83.9 -> 92.1 mm
- net COL1: track 180.2 -> 188.3 mm
- net Net-(D3-A): track 83.6 -> 81.3 mm
- net Net-(D8-A): track 71.1 -> 73.2 mm
- net Net-(D7-A): track 74.4 -> 76.5 mm
- net Net-(D13-A): track 76.2 -> 78.0 mm
- net COL2: track 174.3 -> 175.6 mm
- net Net-(F1-Pad1): track 16.0 -> 15.3 mm
- net COL4: track 104.1 -> 104.7 mm, vias 3 -> 1
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Other:
- board text added: "TEMP"
